Commit message: Release/Flexiv ROS 2 Humble v1.4 (#37)

File: flexiv_description/urdf/flexiv_arm.materials.xacro (robot description, xacro)
@@ -1,7 +1,4 @@
 <?xml version="1.0" ?>
 <robot xmlns:xacro="http://www.ros.org/wiki/xacro">
-    <material name="rizon_blue">
-      <color rgba="0.0 0.0 1.0 0.5"/>
-    </material>
     <material name="rizon_light_grey">
       <color rgba="0.7 0.7 0.7 1.0"/>

File: flexiv_description/urdf/rizon.urdf.xacro (robot description, xacro)
@@ -3,5 +3,5 @@
   <!-- Enable setting arguments from the launch file -->
   <xacro:arg name="name" default="rizon"/>
-  <!-- 'rizon_type' values: rizon4, rizon4s, rizon10 -->
+  <!-- 'rizon_type' values: rizon4, rizon4s, rizon10, rizon10s -->
   <xacro:arg name="rizon_type" default="rizon4"/>
   <!-- import main macro -->
@@ -9,6 +9,5 @@
   <!-- parameters -->
   <xacro:arg name="prefix" default="" />
-  <xacro:arg name="robot_ip" default="" />
-  <xacro:arg name="local_ip" default="" />
+  <xacro:arg name="robot_sn" default="" />
   <xacro:arg name="use_fake_hardware" default="false" />
   <xacro:arg name="fake_sensor_commands" default="false" />
@@ -19,6 +18,5 @@
     rizon_type="$(arg rizon_type)"
     prefix="$(arg prefix)"
-    robot_ip="$(arg robot_ip)"
-    local_ip="$(arg local_ip)"
+    robot_sn="$(arg robot_sn)"
     use_fake_hardware="$(arg use_fake_hardware)"
     fake_sensor_commands="$(arg fake_sensor_commands)"

File: flexiv_description/urdf/rizon10.ros2_control.xacro (robot description, xacro)
@@ -3,6 +3,5 @@
   <xacro:macro name="rizon10_ros2_control" params="
     prefix
-    robot_ip
-    local_ip
+    robot_sn
     use_fake_hardware:=false
     fake_sensor_commands:=false
@@ -18,6 +17,6 @@
         <xacro:unless value="${use_fake_hardware}">
           <plugin>flexiv_hardware/FlexivHardwareInterface</plugin>
-          <param name="robot_ip">${robot_ip}</param>
-          <param name="local_ip">${local_ip}</param>
+          <param name="robot_sn">${robot_sn}</param>
+          <param name="prefix">${prefix}</param>
         </xacro:unless>
       </hardware>
@@ -141,37 +140,38 @@
         <state_interface name="effort"/>
       </joint>
-      <sensor name="${prefix}force_torque_sensor">
-        <state_interface name="force.x"/>
-        <state_interface name="force.y"/>
-        <state_interface name="force.z"/>
-        <state_interface name="torque.x"/>
-        <state_interface name="torque.y"/>
-        <state_interface name="torque.z"/>
-      </sensor>
-      <sensor name="${prefix}external_wrench_in_base">
-        <state_interface name="force.x"/>
-        <state_interface name="force.y"/>
-        <state_interface name="force.z"/>
-        <state_interface name="torque.x"/>
-        <state_interface name="torque.y"/>
-        <state_interface name="torque.z"/>
-      </sensor>
-      <sensor name="${prefix}external_wrench_in_tcp">
-        <state_interface name="force.x"/>
-        <state_interface name="force.y"/>
-        <state_interface name="force.z"/>
-        <state_interface name="torque.x"/>
-        <state_interface name="torque.y"/>
-        <state_interface name="torque.z"/>
-      </sensor>
-      <sensor name="${prefix}tcp_pose">
-        <state_interface name="position.x"/>
-        <state_interface name="position.y"/>
-        <state_interface name="position.z"/>
-        <state_interface name="orientation.x"/>
-        <state_interface name="orientation.y"/>
-        <state_interface name="orientation.z"/>
-        <state_interface name="orientation.w"/>
-      </sensor>
+      <gpio name="${prefix}gpio">
+        <command_interface name="digital_output_0"/>
+        <command_interface name="digital_output_1"/>
+        <command_interface name="digital_output_2"/>
+        <command_interface name="digital_output_3"/>
+        <command_interface name="digital_output_4"/>
+        <command_interface name="digital_output_5"/>
+        <command_interface name="digital_output_6"/>
+        <command_interface name="digital_output_7"/>
+        <command_interface name="digital_output_8"/>
+        <command_interface name="digital_output_9"/>
+        <command_interface name="digital_output_10"/>
+        <command_interface name="digital_output_11"/>
+        <command_interface name="digital_output_12"/>
+        <command_interface name="digital_output_13"/>
+        <command_interface name="digital_output_14"/>
+        <command_interface name="digital_output_15"/>
+        <state_interface name="digital_input_0"/>
+        <state_interface name="digital_input_1"/>
+        <state_interface name="digital_input_2"/>
+        <state_interface name="digital_input_3"/>
+        <state_interface name="digital_input_4"/>
+        <state_interface name="digital_input_5"/>
+        <state_interface name="digital_input_6"/>
+        <state_interface name="digital_input_7"/>
+        <state_interface name="digital_input_8"/>
+        <state_interface name="digital_input_9"/>
+        <state_interface name="digital_input_10"/>
+        <state_interface name="digital_input_11"/>
+        <state_interface name="digital_input_12"/>
+        <state_interface name="digital_input_13"/>
+        <state_interface name="digital_input_14"/>
+        <state_interface name="digital_input_15"/>
+      </gpio>
     </ros2_control>
   </xacro:macro>

File: flexiv_description/urdf/rizon10_joints_links.xacro (robot description, xacro)
@@ -2,5 +2,5 @@
 <robot xmlns:xacro="http://www.ros.org/wiki/xacro">
   <!--
-    rizon_type = "rizon10"
+    rizon_type = "rizon10", "rizon10s"
     prefix = "", "left_"
     mesh_prefix_path = "", "package://flexiv_description/"
@@ -66,5 +66,10 @@
       <parent link="${prefix}link7"/>
       <child link="${prefix}flange"/>
-      <origin xyz="0.0 0.0 0.081" rpy="0 0 ${-pi}"/>
+      <xacro:if value="${rizon_type=='rizon10'}">
+        <origin xyz="0.0 0.0 0.081" rpy="0 0 ${-pi}"/>
+      </xacro:if>
+      <xacro:if value="${rizon_type=='rizon10s'}">
+        <origin xyz="0.0 0.0 0.124" rpy="0 0 ${-pi}"/>
+      </xacro:if>
     </joint>
     <!-- LINKS -->
@@ -77,5 +82,5 @@
         <inertia ixx="0.08" ixy="0.0" ixz="-0.0003" iyy="0.08" iyz="0.001" izz="0.04" />
       </inertial>
-      <visual>
+      <visual name="shell">
         <origin xyz="0 0 0" rpy="0 0 0"/>
         <geometry>
@@ -84,5 +89,5 @@
         <material name="rizon_dark_grey" />
       </visual>
-      <collision>
+      <collision name="hull">
         <origin xyz="0 0 0" rpy="0 0 0"/>
         <geometry>
@@ -97,5 +102,5 @@
         <inertia ixx="0.18" ixy="0.0002" ixz="0.0001" iyy="0.17" iyz="0.02" izz="0.04" />
       </inertial>
-      <visual>
+      <visual name="shell">
         <origin xyz="0 0 0" rpy="0 0 0" />
         <geometry>
@@ -104,5 +109,12 @@
         <material name="rizon_dark_grey" />
       </visual>
-      <collision>
+      <visual name="ring">
+        <origin rpy="0 0 0" xyz="0 0 -0.0025" />
+        <geometry>
+          <mesh filename="${mesh_prefix_path}meshes/${rizon_type}/visual/ring.obj" scale="0.079 0.079 0.002" />
+        </geometry>
+        <material name="rizon_white" />
+      </visual>
+      <collision name="hull">
         <origin xyz="0 0 0" rpy="0 0 0" />
         <geometry>
@@ -117,5 +129,5 @@
         <inertia ixx="0.1" ixy="0.0" ixz="0.0001" iyy="0.08" iyz="0.02" izz="0.03" />
       </inertial>
-      <visual>
+      <visual name="shell">
         <origin xyz="0 0 0" rpy="0 0 0"/>
         <geometry>
@@ -124,5 +136,12 @@
         <material name="rizon_dark_grey" />
       </visual>
-      <collision>
+      <visual name="ring">
+        <origin rpy="1.5707963 0 0" xyz="0 -0.0025 0" />
+        <geometry>
+          <mesh filename="${mesh_prefix_path}meshes/${rizon_type}/visual/ring.obj" scale="0.079 0.079 0.002" />
+        </geometry>
+        <material name="rizon_white" />
+      </visual>
+      <collision name="hull">
         <origin xyz="0 0 0" rpy="0 0 0"/>
         <geometry>
@@ -137,5 +156,5 @@
         <inertia ixx="0.03" ixy="-0.0001" ixz="-0.0001" iyy="0.03" iyz="-0.006" izz="0.01" />
       </inertial>
-      <visual>
+      <visual name="shell">
         <origin xyz="0 0 0" rpy="0 0 0" />
         <geometry>
@@ -144,5 +163,12 @@
         <material name="rizon_dark_grey" />
       </visual>
-      <collision>
+      <visual name="ring">
+        <origin rpy="0 0 0" xyz="0 0 -0.0025" />
+        <geometry>
+          <mesh filename="${mesh_prefix_path}meshes/${rizon_type}/visual/ring.obj" scale="0.062 0.062 0.002" />
+        </geometry>
+        <material name="rizon_white" />
+      </visual>
+      <collision name="hull">
         <origin xyz="0 0 0" rpy="0 0 0" />
         <geometry>
@@ -157,5 +183,5 @@
         <inertia ixx="0.03" ixy="0.0" ixz="-0.0001" iyy="0.03" iyz="0.0007" izz="0.005" />
       </inertial>
-      <visual>
+      <visual name="shell">
         <origin xyz="0 0 0" rpy="0 0 0"/>
         <geometry>
@@ -164,5 +190,12 @@
         <material name="rizon_dark_grey" />
       </visual>
-      <collision>
+      <visual name="ring">
+        <origin rpy="1.5707963 0 0" xyz="0 -0.0025 0" />
+        <geometry>
+          <mesh filename="${mesh_prefix_path}meshes/${rizon_type}/visual/ring.obj" scale="0.062 0.062 0.002" />
+        </geometry>
+        <material name="rizon_white" />
+      </visual>
+      <collision name="hull">
         <origin xyz="0 0 0" rpy="0 0 0"/>
         <geometry>
@@ -177,5 +210,5 @@
         <inertia ixx="0.01" ixy="0.0" ixz="0.0" iyy="0.01" iyz="0.001" izz="0.004" />
       </inertial>
-      <visual>
+      <visual name="shell">
         <origin xyz="0 0 0" rpy="0 0 0"/>
         <geometry>
@@ -184,5 +217,12 @@
         <material name="rizon_dark_grey" />
       </visual>
-      <collision>
+      <visual name="ring">
+        <origin rpy="0 0 0" xyz="0 0 -0.0025" />
+        <geometry>
+          <mesh filename="${mesh_prefix_path}meshes/${rizon_type}/visual/ring.obj" scale="0.051 0.051 0.002" />
+        </geometry>
+        <material name="rizon_white" />
+      </visual>
+      <collision name="hull">
         <origin xyz="0 0 0" rpy="0 0 0"/>
         <geometry>
@@ -197,5 +237,5 @@
         <inertia ixx="0.01" ixy="0.0003" ixz="0.001" iyy="0.01" iyz="0.002" izz="0.004" />
       </inertial>
-      <visual>
+      <visual name="shell">
         <origin xyz="0 0 0" rpy="0 0 0"/>
         <geometry>
@@ -204,5 +244,12 @@
         <material name="rizon_dark_grey" />
       </visual>
-      <collision>
+      <visual name="ring">
+        <origin rpy="1.5707963 0 0" xyz="0 -0.0025 0" />
+        <geometry>
+          <mesh filename="${mesh_prefix_path}meshes/${rizon_type}/visual/ring.obj" scale="0.051 0.051 0.002" />
+        </geometry>
+        <material name="rizon_white" />
+      </visual>
+      <collision name="hull">
         <origin xyz="0 0 0" rpy="0 0 0"/>
         <geometry>
@@ -212,22 +259,58 @@
     </link>
     <link name="${prefix}link7">
-      <inertial>
-        <mass value="0.9" />
-        <origin rpy="0 0 0" xyz="0.0 -0.0 0.03" />
-        <inertia ixx="0.001" ixy="0.0" ixz="0.0" iyy="0.001" iyz="0.0" izz="0.001" />
-      </inertial>
-      <visual>
-        <origin xyz="0 0 0" rpy="0 0 0"/>
-        <geometry>
-          <mesh filename="${mesh_prefix_path}meshes/${rizon_type}/visual/link7.obj" />
-        </geometry>
-        <material name="rizon_dark_grey" />
-      </visual>
-      <collision>
-        <origin xyz="0 0 0" rpy="0 0 0"/>
-        <geometry>
-          <mesh filename="${mesh_prefix_path}meshes/${rizon_type}/collision/link7.stl" />
-        </geometry>
-      </collision>
+      <xacro:if value="${rizon_type=='rizon10'}">
+        <inertial>
+          <mass value="0.9" />
+          <origin rpy="0 0 0" xyz="0.0 -0.0 0.03" />
+          <inertia ixx="0.001" ixy="0.0" ixz="0.0" iyy="0.001" iyz="0.0" izz="0.001" />
+        </inertial>
+        <visual name="shell">
+          <origin xyz="0 0 0" rpy="0 0 0"/>
+          <geometry>
+            <mesh filename="${mesh_prefix_path}meshes/${rizon_type}/visual/link7.obj" />
+          </geometry>
+          <material name="rizon_dark_grey" />
+        </visual>
+        <visual name="ring">
+          <origin rpy="0 0 0" xyz="0 0 -0.0025" />
+          <geometry>
+            <mesh filename="${mesh_prefix_path}meshes/rizon10/visual/ring.obj" scale="0.051 0.051 0.002" />
+          </geometry>
+          <material name="rizon_white" />
+        </visual>
+        <collision name="hull">
+          <origin xyz="0 0 0" rpy="0 0 0"/>
+          <geometry>
+            <mesh filename="${mesh_prefix_path}meshes/${rizon_type}/collision/link7.stl" />
+          </geometry>
+        </collision>
+      </xacro:if>
+      <xacro:if value="${rizon_type=='rizon10s'}">
+        <inertial>
+          <mass value="1.5" />
+          <origin rpy="0 0 0" xyz="0.0 -0.0 0.05" />
+          <inertia ixx="0.001" ixy="0.0" ixz="0.0" iyy="0.001" iyz="0.0" izz="0.001" />
+        </inertial>
+        <visual name="shell">
+          <origin xyz="0 0 0" rpy="0 0 0"/>
+          <geometry>
+            <mesh filename="${mesh_prefix_path}meshes/${rizon_type}/visual/link7.obj" />
+          </geometry>
+          <material name="rizon_dark_grey" />
+        </visual>
+        <visual name="ring">
+          <origin rpy="0 0 0" xyz="0 0 -0.0025" />
+          <geometry>
+            <mesh filename="${mesh_prefix_path}meshes/rizon10/visual/ring.obj" scale="0.051 0.051 0.002" />
+          </geometry>
+          <material name="rizon_white" />
+        </visual>
+        <collision name="hull">
+          <origin xyz="0 0 0" rpy="0 0 0"/>
+          <geometry>
+            <mesh filename="${mesh_prefix_path}meshes/${rizon_type}/collision/link7.stl" />
+          </geometry>
+        </collision>
+      </xacro:if>
     </link>
     <link name="${prefix}flange"/>

File: flexiv_description/urdf/rizon4.ros2_control.xacro (robot description, xacro)
@@ -3,6 +3,5 @@
   <xacro:macro name="rizon4_ros2_control" params="
     prefix
-    robot_ip
-    local_ip
+    robot_sn
     use_fake_hardware:=false
     fake_sensor_commands:=false
@@ -18,6 +17,5 @@
         <xacro:unless value="${use_fake_hardware}">
           <plugin>flexiv_hardware/FlexivHardwareInterface</plugin>
-          <param name="robot_ip">${robot_ip}</param>
-          <param name="local_ip">${local_ip}</param>
+          <param name="robot_sn">${robot_sn}</param>
           <param name="prefix">${prefix}</param>
         </xacro:unless>
@@ -142,37 +140,4 @@
         <state_interface name="effort"/>
       </joint>
-      <sensor name="${prefix}force_torque_sensor">
-        <state_interface name="force.x"/>
-        <state_interface name="force.y"/>
-        <state_interface name="force.z"/>
-        <state_interface name="torque.x"/>
-        <state_interface name="torque.y"/>
-        <state_interface name="torque.z"/>
-      </sensor>
-      <sensor name="${prefix}external_wrench_in_base">
-        <state_interface name="force.x"/>
-        <state_interface name="force.y"/>
-        <state_interface name="force.z"/>
-        <state_interface name="torque.x"/>
-        <state_interface name="torque.y"/>
-        <state_interface name="torque.z"/>
-      </sensor>
-      <sensor name="${prefix}external_wrench_in_tcp">
-        <state_interface name="force.x"/>
-        <state_interface name="force.y"/>
-        <state_interface name="force.z"/>
-        <state_interface name="torque.x"/>
-        <state_interface name="torque.y"/>
-        <state_interface name="torque.z"/>
-      </sensor>
-      <sensor name="${prefix}tcp_pose">
-        <state_interface name="position.x"/>
-        <state_interface name="position.y"/>
-        <state_interface name="position.z"/>
-        <state_interface name="orientation.x"/>
-        <state_interface name="orientation.y"/>
-        <state_interface name="orientation.z"/>
-        <state_interface name="orientation.w"/>
-      </sensor>
       <gpio name="${prefix}gpio">
         <command_interface name="digital_output_0"/>

File: flexiv_description/urdf/rizon4_joints_links.xacro (robot description, xacro)
@@ -59,5 +59,5 @@
       <parent link="${prefix}link6"/>
       <child link="${prefix}link7"/>
-      <origin xyz="-0.055 0.070 0.11" rpy="0 ${-pi/2} 0"/>
+      <origin xyz="-0.015 0.073 0.11" rpy="0 ${-pi/2} 0"/>
       <axis xyz="0 0 1"/>
       <limit effort="39" lower="-2.9671" upper="2.9671" velocity="4.8869" />
@@ -82,5 +82,5 @@
         <inertia ixx="0.02" ixy="0.0" ixz="0.0" iyy="0.02" iyz="0.0001" izz="0.009" />
       </inertial>
-      <visual>
+      <visual name="shell">
         <origin xyz="0 0 0" rpy="0 0 0"/>
         <geometry>
@@ -89,5 +89,5 @@
         <material name="rizon_light_grey" />
       </visual>
-      <collision>
+      <collision name="hull">
         <origin xyz="0 0 0" rpy="0 0 0"/>
         <geometry>
@@ -102,5 +102,5 @@
         <inertia ixx="0.03" ixy="0.0" ixz="0.0" iyy="0.03" iyz="0.002" izz="0.008" />
       </inertial>
-      <visual>
+      <visual name="shell">
         <origin xyz="0 0 0" rpy="0 0 0" />
         <geometry>
@@ -109,5 +109,12 @@
         <material name="rizon_light_grey" />
       </visual>
-      <collision>
+      <visual name="ring">
+        <origin rpy="0 0 0" xyz="0 0 -0.0025" />
+        <geometry>
+          <mesh filename="${mesh_prefix_path}meshes/${rizon_type}/visual/ring.obj" scale="0.062 0.062 0.002" />
+        </geometry>
+        <material name="rizon_white" />
+      </visual>
+      <collision name="hull">
         <origin xyz="0 0 0" rpy="0 0 0" />
         <geometry>
@@ -122,5 +129,5 @@
         <inertia ixx="0.02" ixy="0.0" ixz="0.0" iyy="0.02" iyz="-0.0003" izz="0.004" />
       </inertial>
-      <visual>
+      <visual name="shell">
         <origin xyz="0 0 0" rpy="0 0 0"/>
         <geometry>
@@ -129,5 +136,12 @@
         <material name="rizon_light_grey" />
       </visual>
-      <collision>
+      <visual name="ring">
+        <origin rpy="${pi/2} 0 0" xyz="0 -0.0025 0" />
+        <geometry>
+          <mesh filename="${mesh_prefix_path}meshes/${rizon_type}/visual/ring.obj" scale="0.062 0.062 0.002" />
+        </geometry>
+        <material name="rizon_white" />
+      </visual>
+      <collision name="hull">
         <origin xyz="0 0 0" rpy="0 0 0"/>
         <geometry>
@@ -142,5 +156,5 @@
         <inertia ixx="0.01" ixy="0.00" ixz="-0.001" iyy="0.01" iyz="-0.0007" izz="0.004" />
       </inertial>
-      <visual>
+      <visual name="shell">
         <origin xyz="0 0 0" rpy="0 0 0" />
         <geometry>
@@ -149,5 +163,12 @@
         <material name="rizon_light_grey" />
       </visual>
-      <collision>
+      <visual name="ring">
+        <origin rpy="0 0 0" xyz="0 0 -0.0025" />
+        <geometry>
+          <mesh filename="${mesh_prefix_path}meshes/${rizon_type}/visual/ring.obj" scale="0.051 0.051 0.002" />
+        </geometry>
+        <material name="rizon_white" />
+      </visual>
+      <collision name="hull">
         <origin xyz="0 0 0" rpy="0 0 0" />
         <geometry>
@@ -162,5 +183,5 @@
         <inertia ixx="0.02" ixy="0.00" ixz="-0.002" iyy="0.02" iyz="-0.001" izz="0.003" />
       </inertial>
-      <visual>
+      <visual name="shell">
         <origin xyz="0 0 0" rpy="0 0 0"/>
         <geometry>
@@ -169,5 +190,12 @@
         <material name="rizon_light_grey" />
       </visual>
-      <collision>
+      <visual name="ring">
+        <origin rpy="${pi/2} 0 0" xyz="0 -0.0025 0" />
+        <geometry>
+          <mesh filename="${mesh_prefix_path}meshes/${rizon_type}/visual/ring.obj" scale="0.051 0.051 0.002" />
+        </geometry>
+        <material name="rizon_white" />
+      </visual>
+      <collision name="hull">
         <origin xyz="0 0 0" rpy="0 0 0"/>
         <geometry>
@@ -182,5 +210,5 @@
         <inertia ixx="0.01" ixy="0.0" ixz="0.0" iyy="0.01" iyz="0.001" izz="0.004" />
       </inertial>
-      <visual>
+      <visual name="shell">
         <origin xyz="0 0 0" rpy="0 0 0"/>
         <geometry>
@@ -189,5 +217,12 @@
         <material name="rizon_light_grey" />
       </visual>
-      <collision>
+      <visual name="ring">
+        <origin rpy="0 0 0" xyz="0 0 -0.0025" />
+        <geometry>
+          <mesh filename="${mesh_prefix_path}meshes/${rizon_type}/visual/ring.obj" scale="0.051 0.051 0.002" />
+        </geometry>
+        <material name="rizon_white" />
+      </visual>
+      <collision name="hull">
         <origin xyz="0 0 0" rpy="0 0 0"/>
         <geometry>
@@ -202,5 +237,5 @@
         <inertia ixx="0.01" ixy="-0.000" ixz="-0.001" iyy="0.01" iyz="0.002" izz="0.004" />
       </inertial>
-      <visual>
+      <visual name="shell">
         <origin xyz="0 0 0" rpy="0 0 0"/>
         <geometry>
@@ -209,5 +244,12 @@
         <material name="rizon_light_grey" />
       </visual>
-      <collision>
+      <visual name="ring">
+        <origin rpy="${pi/2} 0 0" xyz="0 -0.0025 0" />
+        <geometry>
+          <mesh filename="${mesh_prefix_path}meshes/${rizon_type}/visual/ring.obj" scale="0.051 0.051 0.002" />
+        </geometry>
+        <material name="rizon_white" />
+      </visual>
+      <collision name="hull">
         <origin xyz="0 0 0" rpy="0 0 0"/>
         <geometry>
@@ -223,5 +265,5 @@
           <inertia ixx="0.001" ixy="0.0" ixz="0.0" iyy="0.001" iyz="0.0" izz="0.001" />
         </inertial>
-        <visual>
+        <visual name="shell">
           <origin xyz="0 0 0" rpy="0 0 0"/>
           <geometry>
@@ -230,5 +272,12 @@
           <material name="rizon_light_grey" />
         </visual>
-        <collision>
+        <visual name="ring">
+          <origin rpy="0 0 0" xyz="0 0 -0.0025" />
+          <geometry>
+            <mesh filename="${mesh_prefix_path}meshes/${rizon_type}/visual/ring.obj" scale="0.051 0.051 0.002" />
+          </geometry>
+          <material name="rizon_white" />
+        </visual>
+        <collision name="hull">
           <origin xyz="0 0 0" rpy="0 0 0"/>
           <geometry>
@@ -243,5 +292,5 @@
           <inertia ixx="0.001" ixy="0.0" ixz="0.0" iyy="0.001" iyz="0.0" izz="0.001" />
         </inertial>
-        <visual>
+        <visual name="shell">
           <origin xyz="0 0 0" rpy="0 0 0"/>
           <geometry>
@@ -250,5 +299,12 @@
           <material name="rizon_light_grey" />
         </visual>
-        <collision>
+        <visual name="ring">
+          <origin rpy="0 0 0" xyz="0 0 -0.0025" />
+          <geometry>
+            <mesh filename="${mesh_prefix_path}meshes/${rizon_type}/visual/ring.obj" scale="0.051 0.051 0.002" />
+          </geometry>
+          <material name="rizon_white" />
+        </visual>
+        <collision name="hull">
           <origin xyz="0 0 0" rpy="0 0 0"/>
           <geometry>
