Commit message: Release/Flexiv ROS 2 Humble v1.4 (#37)

File: flexiv_description/urdf/rizon_macro.xacro (robot description, xacro)
@@ -4,6 +4,5 @@
     rizon_type
     prefix
-    robot_ip
-    local_ip
+    robot_sn
     use_fake_hardware:=false
     fake_sensor_commands:=false
@@ -18,18 +17,18 @@
       <!-- ros2 control include -->
       <xacro:include filename="$(find flexiv_description)/urdf/rizon4.ros2_control.xacro"/>
-      <xacro:rizon4_ros2_control prefix="${prefix}" robot_ip="${robot_ip}"
-        local_ip="${local_ip}" use_fake_hardware="${use_fake_hardware}"
+      <xacro:rizon4_ros2_control prefix="${prefix}" robot_sn="${robot_sn}"
+        use_fake_hardware="${use_fake_hardware}"
         fake_sensor_commands="${fake_sensor_commands}"
         initial_positions="${initial_positions}"
         />
     </xacro:if>
-    <!-- Rizon 10 -->
-    <xacro:if value="${rizon_type=='rizon10'}">
+    <!-- Rizon 10 or 10s-->
+    <xacro:if value="${rizon_type=='rizon10' or rizon_type=='rizon10s'}">
       <xacro:include filename="$(find flexiv_description)/urdf/rizon10_joints_links.xacro" />
       <xacro:rizon10_joints_links rizon_type="${rizon_type}" prefix="${prefix}" mesh_prefix_path="package://flexiv_description/" />
       <!-- ros2 control include -->
       <xacro:include filename="$(find flexiv_description)/urdf/rizon10.ros2_control.xacro"/>
-      <xacro:rizon10_ros2_control prefix="${prefix}" robot_ip="${robot_ip}"
-        local_ip="${local_ip}" use_fake_hardware="${use_fake_hardware}"
+      <xacro:rizon10_ros2_control prefix="${prefix}" robot_sn="${robot_sn}"
+        use_fake_hardware="${use_fake_hardware}"
         fake_sensor_commands="${fake_sensor_commands}"
         initial_positions="${initial_positions}"
